File: hard/Bottom.kicad_pcb (KiCad board)
At the start: 2 copper layers, 105 x 195 mm, 0 parts

Commit message: modify for rev 1.1
Routing:
- removed copper zone on B.Cu, net +3.3V
- removed copper zone on F.Cu, net GND
- removed copper zone on B.Cu, net VBUS
- removed copper zone on F.Cu, net VBUS
Other:
- outline, holes or cut-outs redrawn
Changed lines of the file:
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@@
 	)
 	(net 0 "")
-	(net 1 "GND")
-	(net 2 "+3.3V")
-	(net 3 "VBUS")
 	(gr_circle
 		(center 58 46)
@@
 	)
 	(gr_circle
+		(center 155 149)
+		(end 156.6 149)
+		(stroke
+			(width 0.05)
+			(type default)
+		)
+		(fill none)
+		(layer "Edge.Cuts")
+	)
+	(gr_circle
 		(center 155 233)
 		(end 156.6 233)
@@
 			(type default)
 		)
+		(layer "Edge.Cuts")
+	)
+	(gr_circle
+		(center 58 149)
+		(end 59.6 149)
+		(stroke
+			(width 0.05)
+			(type default)
+		)
+		(fill none)
 		(layer "Edge.Cuts")
 	)
@@
 			(extension_offset 0.5) keep_text_aligned)
 	)
-	(zone
-		(net 1)
-		(net_name "GND")
-		(layer "F.Cu")
-		(hatch edge 0.5)
-		(priority 100)
-		(connect_pads
-			(clearance 0.5)
-		)
-		(min_thickness 0.25)
-		(filled_areas_thickness no)
-		(fill yes
-			(thermal_gap 0.5)
-			(thermal_bridge_width 0.5)
-		)
-		(polygon
-			(pts
-				(xy 54 42) (xy 159 42) (xy 159 237) (xy 54 237)
-			)
-		)
-	)
-	(zone
-		(net 3)
-		(net_name "VBUS")
-		(layer "F.Cu")
-		(hatch edge 0.5)
-		(connect_pads
-			(clearance 0.5)
-		)
-		(min_thickness 0.25)
-		(filled_areas_thickness no)
-		(fill yes
-			(thermal_gap 0.5)
-			(thermal_bridge_width 0.5)
-		)
-		(polygon
-			(pts
-				(xy 54 42) (xy 159 42) (xy 159 237) (xy 54 237)
-			)
-		)
-	)
-	(zone
-		(net 2)
-		(net_name "+3.3V")
-		(layer "B.Cu")
-		(hatch edge 0.5)
-		(priority 100)
-		(connect_pads
-			(clearance 0.5)
-		)
-		(min_thickness 0.25)
-		(filled_areas_thickness no)
-		(fill yes
-			(thermal_gap 0.5)
-			(thermal_bridge_width 0.5)
-		)
-		(polygon
-			(pts
-				(xy 54 42) (xy 159 42) (xy 159 237) (xy 54 237)
-			)
-		)
-	)
-	(zone
-		(net 3)
-		(net_name "VBUS")
-		(layer "B.Cu")
-		(hatch edge 0.5)
-		(priority 1)
-		(connect_pads
-			(clearance 0.5)
-		)
-		(min_thickness 0.25)
-		(filled_areas_thickness no)
-		(fill yes
-			(thermal_gap 0.5)
-			(thermal_bridge_width 0.5)
-		)
-		(polygon
-			(pts
-				(xy 54 42) (xy 159 42) (xy 159 237) (xy 54 237)
-			)
-		)
-	)
 )
