File: hard/Case_acrylic.kicad_pcb (KiCad board)
At the start: 2 copper layers, 105 x 195 mm, 0 parts

Commit message: modify for rev 1.1
Other:
- outline, holes or cut-outs redrawn
Changed lines of the file:
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@@
 				(thickness 0.035)
 			)
-			(layer "dielectric 1"
+			(layer "dielectric 2"
 				(type "core")
 				(thickness 1.51)
@@
 	)
 	(gr_circle
+		(center 58 149)
+		(end 59.6 149)
+		(stroke
+			(width 0.05)
+			(type default)
+		)
+		(fill none)
+		(layer "Edge.Cuts")
+	)
+	(gr_circle
 		(center 117.5 140.06336)
 		(end 120.7 140.06336)
@@
 		(stroke
 			(width 0.05)
+			(type default)
+		)
+		(fill none)
+		(layer "Edge.Cuts")
+	)
+	(gr_circle
+		(center 155 149)
+		(end 156.6 149)
+		(stroke
+			(width 0.05)
